Commit message: [hardware_interface] under construct

File: configuration/ar/ros2_control/ar.ros2_control.xacro (robot description, xacro)
@@ -1,9 +1,8 @@
 <?xml version="1.0"?>
 <robot xmlns:xacro="http://www.ros.org/wiki/xacro">
-  <xacro:macro name="ar_control" params="name desc sim ui">
+  <xacro:macro name="ar_control" params="name sim ui">
     <ros2_control name="${name}" type="system">
       <hardware>
         <plugin>ar_control/ArSystemHardware</plugin>
-        <param name="desc">${desc}</param>
         <param name="sim">${sim}</param>
         <param name="ui">${ui}</param>
