Commit message: [ar_planner] update launch file can plan with 2 pipeline ompl and pilz

File: ar_src/configuration/ar/config/ar_config.srdf.xacro (robot description, xacro)
@@ -7,10 +7,11 @@
 	<!--SUBGROUPS: Groups can also be formed by referencing to already defined group names-->
 	<group name="Arm">
-		<joint name="Arm_joint1" />
-		<joint name="Arm_joint2" />
-		<joint name="Arm_joint3" />
-		<joint name="Arm_joint4" />
-		<joint name="Arm_joint5" />
-		<joint name="Arm_joint6" />
+		<joint name="Arm_joint1"/>
+		<joint name="Arm_joint2"/>
+		<joint name="Arm_joint3"/>
+		<joint name="Arm_joint4"/>
+		<joint name="Arm_joint5"/>
+		<joint name="Arm_joint6"/>
+		<joint name="Arm_eejoint"/>
 	</group>
 	<!--GROUP STATES: Purpose: Define a named state for a particular group, in terms of joint values. This is useful to define states like 'folded Arms'-->
@@ -42,3 +43,5 @@
 	<disable_collisions link1="Arm_link4" link2="Arm_link5" reason="Adjacent" />
 	<disable_collisions link1="Arm_link5" link2="Arm_endlink" reason="Adjacent" />
+	<disable_collisions link1="Arm_endlink" link2="Arm_eelink" reason="Adjacent" />
+	<disable_collisions link1="Arm_link5" link2="Arm_eelink" reason="Adjacent" />
 </robot>

File: ar_src/configuration/ar/urdf/ar_base.xacro (robot description, xacro)
@@ -4,232 +4,208 @@
      For more information, please see http://wiki.ros.org/sw_urdf_exporter -->
 <robot name="ar"
-	xmlns:xacro="http://www.ros.org/wiki/xacro">
-	<link name = "world"/>
-	<link name="Base">
-		<visual>
-			<geometry>
-				<mesh filename="package://ar_moveit_config/meshes/visuals/base_link.STL"/>
-			</geometry>
-			<origin xyz="0 0 0" rpy="0 0 0"/>
-			<material name="">
-				<color rgba="0.6 0.6 0.6 1" />
-			</material>
-		</visual>
-		<collision>
-			<geometry>
-				<mesh filename="package://ar_moveit_config/meshes/collisions/base_link.STL"/>
-			</geometry>
-			<origin xyz="0 0 0" rpy="0 0 0"/>
-		</collision>
-	</link>
-	<joint name = "Base_joint" type ="fixed">
-		<parent link = "world"/>
-		<child link = "Base"/>
-		<origin xyz="0 0 0" rpy="0 0 0"/>
-	</joint>
-	<link name="Arm_link1">
-		<inertial>
-        	<origin rpy="0 0 0" xyz="-0.022706 0.04294 -0.12205"/>
-        	<mass value="0.88065"/>
-        	<inertia ixx="0.0034" ixy="0.00042296" ixz="-0.00089231" iyy="0.0041778" iyz="0.0010848" izz="0.0027077"/>
-      	</inertial>
-		<visual>
-        	<origin rpy="0 0 0" xyz="0 0 0"/>
-        	<geometry>
-          		<mesh filename="package://ar_moveit_config/meshes/visuals/link_1.STL"/>
-        	</geometry>
-        	<material name="">
-          		<color rgba="0.6 0.6 0.6 1"/>
-        	</material>
-      	</visual>
-		<collision>
-        	<origin rpy="0 0 0" xyz="0 0 0"/>
-        	<geometry>
-          		<mesh filename="package://ar_moveit_config/meshes/collisions/link_1.STL"/>
-        	</geometry>
-      	</collision>
-	</link>
-	<joint name="Arm_joint1" type="revolute">
-    	<origin rpy="3.1415 0 0" xyz="0 0 0"/>
-    	<parent link="Base"/>
-    	<child link="Arm_link1"/>
-    	<axis xyz="0 0 1"/>
-    	<limit
-        	lower="-2.967059728"
-        	upper="2.967059728"
-    		effort="1000"
-        	velocity="1.0472"
-    	/>
-    </joint>
-	<link name="Arm_link2">
-      <inertial>
-        <origin rpy="0 0 0" xyz="0.064818 -0.11189 -0.038671"/>
-        <mass value="0.57738"/>
-        <inertia ixx="0.0047312" ixy="0.0022624" ixz="0.00032144" iyy="0.0020836" iyz="-0.00056569" izz="0.0056129"/>
-      </inertial>
-      <visual>
-        <origin rpy="0 0 0" xyz="0 0 0"/>
-        <geometry>
-          <mesh filename="package://ar_moveit_config/meshes/visuals/link_2.STL"/>
-        </geometry>
-        <material name="">
-          <color rgba="0.6 0.6 0.6 1"/>
-        </material>
-      </visual>
-      <collision>
-        <origin rpy="0 0 0" xyz="0 0 0"/>
-        <geometry>
-          <mesh filename="package://ar_moveit_config/meshes/collisions/link_2.STL"/>
-        </geometry>
-      </collision>
-    </link>
-    <joint name="Arm_joint2" type="revolute">
-    	<origin rpy="1.5708 0 -1.5708" xyz="0 0.0642 -0.16977"/>
-    	<parent link="Arm_link1"/>
-    	<child link="Arm_link2"/>
-    	<axis xyz="0 0 -1"/>
-    	<limit
-        	lower="-0.733038286"
-        	upper="1.5708"
-        	effort="1000"
-        	velocity="1.0472"
-    	/>
-    </joint>
-    <link name="Arm_link3">
-      <inertial>
-        <origin rpy="0 0 0" xyz="-0.00029765 -0.023661 -0.0019125"/>
-        <mass value="0.1787"/>
-        <inertia ixx="0.0001685" ixy="-2.7713E-05" ixz="5.6885E-06" iyy="0.00012865" iyz="2.9256E-05" izz="0.00020744"/>
-      </inertial>
-      <visual>
-        <origin rpy="0 0 0" xyz="0 0 0"/>
-        <geometry>
-          <mesh filename="package://ar_moveit_config/meshes/visuals/link_3.STL"/>
-        </geometry>
-        <material name="">
-          <color rgba="0.6 0.6 0.6 1"/>
-        </material>
-      </visual>
-      <collision>
-        <origin rpy="0 0 0" xyz="0 0 0"/>
-        <geometry>
-          <mesh filename="package://ar_moveit_config/meshes/collisions/link_3.STL"/>
-        </geometry>
-      </collision>
-    </link>
-    <joint name="Arm_joint3" type="revolute">
-      <origin rpy="0 0 3.1416" xyz="0 -0.305 0.007"/>
-      <parent link="Arm_link2"/>
-      <child link="Arm_link3"/>
-      <axis xyz="0 0 -1"/>
-      <limit
-        lower="-1.5533"
-        upper="0.9076"
-        effort="1000"
-        velocity="1.0472"
-      />
-    </joint>
-    <link name="Arm_link4">
-      <inertial>
-        <origin rpy="0 0 0" xyz="-0.0016798 -0.00057319 -0.074404"/>
-        <mass value="0.34936"/>
-        <inertia ixx="0.0030532" ixy="-1.8615E-05" ixz="-7.0047E-05" iyy="0.0031033" iyz="-2.3301E-05" izz="0.00022264"/>
-      </inertial>
-      <visual>
-        <origin rpy="0 0 0" xyz="0 0 0"/>
-        <geometry>
-          <mesh filename="package://ar_moveit_config/meshes/visuals/link_4.STL"/>
-        </geometry>
-        <material name="">
-          <color rgba="0.6 0.6 0.6 1"/>
-        </material>
-      </visual>
-      <collision>
-        <origin rpy="0 0 0" xyz="0 0 0"/>
-        <geometry>
-          <mesh filename="package://ar_moveit_config/meshes/collisions/link_4.STL"/>
-        </geometry>
-      </collision>
-    </link>
-    <joint name="Arm_joint4" type="revolute">
-      <origin rpy="1.5708 0 -1.5708" xyz="0 0 0.0"/>
-      <parent link="Arm_link3"/>
-      <child link="Arm_link4"/>
-      <axis xyz="0 0 -1"/>
-      <limit
-        lower="-3.14159"
-        upper="3.14159"
-        effort="1000"
-        velocity="1.0472"
-      />
-    </joint>
-    <link name="Arm_link5">
-      <inertial>
-        <origin rpy="0 0 0" xyz="0.0015066 -1.3102E-05 -0.012585"/>
-        <mass value="0.11562"/>
-        <inertia ixx="5.5035E-05" ixy="-1.019E-08" ixz="-2.6243E-06" iyy="8.2921E-05" iyz="1.4437E-08" izz="5.2518E-05"/>
-      </inertial>
-      <visual>
-        <origin rpy="0 0 0" xyz="0 0 0"/>
-        <geometry>
-          <mesh filename="package://ar_moveit_config/meshes/visuals/link_5.STL"/>
-        </geometry>
-        <material name="">
-          <color rgba="0.6 0.6 0.6 1"/>
-        </material>
-      </visual>
-      <collision>
-        <origin rpy="0 0 0" xyz="0 0 0"/>
-        <geometry>
-          <mesh filename="package://ar_moveit_config/meshes/collisions/link_5.STL"/>
-        </geometry>
-      </collision>
-    </link>
-    <joint name="Arm_joint5" type="revolute">
-      <origin rpy="3.1415 0 -1.5708" xyz="0 0 -0.22263"/>
-      <parent link="Arm_link4"/>
-      <child link="Arm_link5"/>
-      <axis xyz="1 0 0"/>
-      <limit
-        lower="-1.832595715"
-        upper="1.832595715"
-        effort="1000"
-        velocity="1.0472"
-      />
-    </joint>
-    <link name="Arm_endlink">
-      <inertial>
-        <origin rpy="0 0 0" xyz="2.9287E-10 -1.6472E-09 0.0091432"/>
-        <mass value="0.013863"/>
-        <inertia ixx="1.3596E-06" ixy="3.0585E-13" ixz="5.7102E-14" iyy="1.7157E-06" iyz="6.3369E-09" izz="2.4332E-06"/>
-      </inertial>
-      <visual>
-        <origin rpy="0 0 0" xyz="0 0 0"/>
-        <geometry>
-          <mesh filename="package://ar_moveit_config/meshes/visuals/link_6.STL"/>
-        </geometry>
-        <material name="">
-          <color rgba="0.6 0.6 0.6 1"/>
-        </material>
-      </visual>
-      <collision>
-        <origin rpy="0 0 0" xyz="0 0 0"/>
-        <geometry>
-          <mesh filename="package://ar_moveit_config/meshes/collisions/link_6.STL"/>
-        </geometry>
-      </collision>
-    </link>
-    <joint name="Arm_joint6" type="revolute">
-      <origin rpy="0 0 3.1416" xyz="0.000 0 0.041"/>
-      <parent link="Arm_link5"/>
-      <child link="Arm_endlink"/>
-      <axis xyz="0 0 1"/>
-      <limit
-        lower="-3.1415"
-        upper="3.1415"
-        effort="1000"
-        velocity="1.0472"
-      />
-    </joint>
-    <!-- center of the end effector mounting surface on link_6 -->
+  xmlns:xacro="http://www.ros.org/wiki/xacro">
+  <link name = "world"/>
+  <link name="Base">
+    <visual>
+      <geometry>
+        <mesh filename="package://ar_moveit_config/meshes/visuals/base_link.STL"/>
+      </geometry>
+      <origin xyz="0 0 0" rpy="0 0 0"/>
+      <material name="">
+        <color rgba="0.6 0.6 0.6 1" />
+      </material>
+    </visual>
+    <collision>
+      <geometry>
+        <mesh filename="package://ar_moveit_config/meshes/collisions/base_link.STL"/>
+      </geometry>
+      <origin xyz="0 0 0" rpy="0 0 0"/>
+    </collision>
+  </link>
+  <joint name = "Base_joint" type ="fixed">
+    <parent link = "world"/>
+    <child link = "Base"/>
+    <origin xyz="0 0 0" rpy="0 0 0"/>
+  </joint>
+  <link name="Arm_link1">
+    <inertial>
+      <origin rpy="0 0 0" xyz="-0.022706 0.04294 -0.12205"/>
+      <mass value="0.88065"/>
+      <inertia ixx="0.0034" ixy="0.00042296" ixz="-0.00089231" iyy="0.0041778" iyz="0.0010848" izz="0.0027077"/>
+    </inertial>
+    <visual>
+      <origin rpy="0 0 0" xyz="0 0 0"/>
+      <geometry>
+        <mesh filename="package://ar_moveit_config/meshes/visuals/link_1.STL"/>
+      </geometry>
+      <material name="">
+        <color rgba="0.6 0.6 0.6 1"/>
+      </material>
+    </visual>
+    <collision>
+      <origin rpy="0 0 0" xyz="0 0 0"/>
+      <geometry>
+        <mesh filename="package://ar_moveit_config/meshes/collisions/link_1.STL"/>
+      </geometry>
+    </collision>
+  </link>
+  <joint name="Arm_joint1" type="revolute">
+    <origin rpy="3.1415 0 0" xyz="0 0 0"/>
+    <parent link="Base"/>
+    <child link="Arm_link1"/>
+    <axis xyz="0 0 1"/>
+    <limit lower="-2.967059728" upper="2.967059728" effort="1000" velocity="1.0472" />
+  </joint>
+  <link name="Arm_link2">
+    <inertial>
+      <origin rpy="0 0 0" xyz="0.064818 -0.11189 -0.038671"/>
+      <mass value="0.57738"/>
+      <inertia ixx="0.0047312" ixy="0.0022624" ixz="0.00032144" iyy="0.0020836" iyz="-0.00056569" izz="0.0056129"/>
+    </inertial>
+    <visual>
+      <origin rpy="0 0 0" xyz="0 0 0"/>
+      <geometry>
+        <mesh filename="package://ar_moveit_config/meshes/visuals/link_2.STL"/>
+      </geometry>
+      <material name="">
+        <color rgba="0.6 0.6 0.6 1"/>
+      </material>
+    </visual>
+    <collision>
+      <origin rpy="0 0 0" xyz="0 0 0"/>
+      <geometry>
+        <mesh filename="package://ar_moveit_config/meshes/collisions/link_2.STL"/>
+      </geometry>
+    </collision>
+  </link>
+  <joint name="Arm_joint2" type="revolute">
+    <origin rpy="1.5708 0 -1.5708" xyz="0 0.0642 -0.16977"/>
+    <parent link="Arm_link1"/>
+    <child link="Arm_link2"/>
+    <axis xyz="0 0 -1"/>
+    <limit lower="-0.733038286" upper="1.5708" effort="1000" velocity="1.0472" />
+  </joint>
+  <link name="Arm_link3">
+    <inertial>
+      <origin rpy="0 0 0" xyz="-0.00029765 -0.023661 -0.0019125"/>
+      <mass value="0.1787"/>
+      <inertia ixx="0.0001685" ixy="-2.7713E-05" ixz="5.6885E-06" iyy="0.00012865" iyz="2.9256E-05" izz="0.00020744"/>
+    </inertial>
+    <visual>
+      <origin rpy="0 0 0" xyz="0 0 0"/>
+      <geometry>
+        <mesh filename="package://ar_moveit_config/meshes/visuals/link_3.STL"/>
+      </geometry>
+      <material name="">
+        <color rgba="0.6 0.6 0.6 1"/>
+      </material>
+    </visual>
+    <collision>
+      <origin rpy="0 0 0" xyz="0 0 0"/>
+      <geometry>
+        <mesh filename="package://ar_moveit_config/meshes/collisions/link_3.STL"/>
+      </geometry>
+    </collision>
+  </link>
+  <joint name="Arm_joint3" type="revolute">
+    <origin rpy="0 0 3.1416" xyz="0 -0.305 0.007"/>
+    <parent link="Arm_link2"/>
+    <child link="Arm_link3"/>
+    <axis xyz="0 0 -1"/>
+    <limit lower="-1.5533" upper="0.9076" effort="1000" velocity="1.0472" />
+  </joint>
+  <link name="Arm_link4">
+    <inertial>
+      <origin rpy="0 0 0" xyz="-0.0016798 -0.00057319 -0.074404"/>
+      <mass value="0.34936"/>
+      <inertia ixx="0.0030532" ixy="-1.8615E-05" ixz="-7.0047E-05" iyy="0.0031033" iyz="-2.3301E-05" izz="0.00022264"/>
+    </inertial>
+    <visual>
+      <origin rpy="0 0 0" xyz="0 0 0"/>
+      <geometry>
+        <mesh filename="package://ar_moveit_config/meshes/visuals/link_4.STL"/>
+      </geometry>
+      <material name="">
+        <color rgba="0.6 0.6 0.6 1"/>
+      </material>
+    </visual>
+    <collision>
+      <origin rpy="0 0 0" xyz="0 0 0"/>
+      <geometry>
+        <mesh filename="package://ar_moveit_config/meshes/collisions/link_4.STL"/>
+      </geometry>
+    </collision>
+  </link>
+  <joint name="Arm_joint4" type="revolute">
+    <origin rpy="1.5708 0 -1.5708" xyz="0 0 0.0"/>
+    <parent link="Arm_link3"/>
+    <child link="Arm_link4"/>
+    <axis xyz="0 0 -1"/>
+    <limit lower="-3.14159" upper="3.14159" effort="1000" velocity="1.0472" />
+  </joint>
+  <link name="Arm_link5">
+    <inertial>
+      <origin rpy="0 0 0" xyz="0.0015066 -1.3102E-05 -0.012585"/>
+      <mass value="0.11562"/>
+      <inertia ixx="5.5035E-05" ixy="-1.019E-08" ixz="-2.6243E-06" iyy="8.2921E-05" iyz="1.4437E-08" izz="5.2518E-05"/>
+    </inertial>
+    <visual>
+      <origin rpy="0 0 0" xyz="0 0 0"/>
+      <geometry>
+        <mesh filename="package://ar_moveit_config/meshes/visuals/link_5.STL"/>
+      </geometry>
+      <material name="">
+        <color rgba="0.6 0.6 0.6 1"/>
+      </material>
+    </visual>
+    <collision>
+      <origin rpy="0 0 0" xyz="0 0 0"/>
+      <geometry>
+        <mesh filename="package://ar_moveit_config/meshes/collisions/link_5.STL"/>
+      </geometry>
+    </collision>
+  </link>
+  <joint name="Arm_joint5" type="revolute">
+    <origin rpy="3.1415 0 -1.5708" xyz="0 0 -0.22263"/>
+    <parent link="Arm_link4"/>
+    <child link="Arm_link5"/>
+    <axis xyz="1 0 0"/>
+    <limit lower="-1.832595715" upper="1.832595715" effort="1000" velocity="1.0472" />
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