Commit message: [ar_system]  add argument ready for igh Ethercat Master implement

File: src/configuration/ar/config/ar_config.urdf.xacro (robot description, xacro)
@@ -3,8 +3,9 @@
 	<xacro:arg name="sim" default="false"/>
 	<xacro:arg name="ui" default="false"/>
+	<xacro:arg name="ecat" default="true"/>
 	<!-- Import ar urdf file -->
 	<xacro:include filename="$(find ar_moveit_config)/urdf/ar_base.xacro" />
 	<!-- Import ar ros2_control description -->
 	<xacro:include filename="$(find ar_moveit_config)/ros2_control/ar.ros2_control.xacro" />
-	<xacro:ar_control name="ArSystem" sim="$(arg sim)" ui="$(arg ui)"/>
+	<xacro:ar_control name="ArSystem" sim="$(arg sim)" ui="$(arg ui)" ecat="$(arg ecat)"/>
 </robot>

File: src/configuration/ar/ros2_control/ar.ros2_control.xacro (robot description, xacro)
@@ -1,5 +1,5 @@
 <?xml version="1.0"?>
 <robot xmlns:xacro="http://www.ros.org/wiki/xacro">
-  <xacro:macro name="ar_control" params="name sim ui">
+  <xacro:macro name="ar_control" params="name sim ui ecat">
     <ros2_control name="${name}" type="system">
       <hardware>
@@ -8,4 +8,5 @@
         <param name="sim">${sim}</param>
         <param name="ui">${ui}</param>
+        <param name="ecat">${ecat}</param>
       </hardware>
     </ros2_control>
